File: EDA/nRF_dev/nRF_dev.kicad_pcb (KiCad board)
At the start: 2 copper layers, 78.2 x 100 mm, 50 parts, among them J1 USB_B_Micro, J10 nRF_DBG, J11 UART, J2 Jack-DC, J3 Micro_SD_Card, J4 Conn_01x08_Male, J5 OV7675_DBG, J6 FH26W-25S-0.3SHW(60), J7 Conn_01x08_Male, J8 Conn_01x15_Male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

Commit message: revision 0.0.3 of the nRF dev board
Parts:
- added D1: LED, LED_SMD:LED_0603_1608Metric_Pad1.05x0.95mm_HandSolder, F.Cu at (55.9, 116.8)
- added R6: 10 kΩ, Resistor_SMD:R_0402_1005Metric, F.Cu at (51.9, 116.1)
- added R8: 10 kΩ, Resistor_SMD:R_0402_1005Metric, F.Cu at (51.9, 117.6)
- added U7: SIP32508DT-T1-GE3, Package_TO_SOT_SMD:SOT-23-6, F.Cu at (82.8, 135.2)
- moved C19 4.02 mm to (83.8, 155.6), turned to -90 degrees
Connections:
- net Net-(J8-Pad4) renamed LED
- J5 pad 15: CB_D0 -> CB_D1
- J5 pad 16: CB_D1 -> CB_D0
- J6 pad 1: unconnected-(J6-Pad1) -> PDN
- J6 pad 10: CB_D6 -> HREF
- J6 pad 11: CB_D7 -> XCLK
- J6 pad 12: SCL -> CB_GND
- J6 pad 14: CB_GND -> SCL
- J6 pad 15: XCLK -> CB_D7
- J6 pad 16: HREF -> CB_D6
- J6 pad 17: PCLK -> CB_D5
- J6 pad 18: CB_GND -> CB_D4
- J6 pad 19: CB_VCC -> CB_D3
- J6 pad 20: CB_VCC -> CB_D2
- J6 pad 21: VS -> CB_D1
- J6 pad 22: unconnected-(J6-Pad22) -> CB_D0
- J6 pad 25: PDN -> unconnected-(J6-Pad25)
- J6 pad 4: CB_D0 -> unconnected-(J6-Pad4)
- J6 pad 5: CB_D1 -> VS
- J6 pad 6: CB_D2 -> CB_VCC
- J6 pad 7: CB_D3 -> CB_VCC
- J6 pad 8: CB_D4 -> CB_GND
- J6 pad 9: CB_D5 -> PCLK
- JP1 pad 3: CB_VIN -> Net-(JP1-Pad3)
- U3 pad 15: CB_VIN -> CB_VEN
- U4 pad 15: CB_D0 -> CB_D1
- U4 pad 16: CB_D1 -> CB_D0
Routing:
- net CB_VIN: track 54.4 -> 0.00 mm
- net CB_VEN: track 0.00 -> 46.2 mm
- net CB_VCC: track 57.5 -> 25.9 mm, vias 2 -> 0
- net LED: track 76.9 -> 99.8 mm
- net PDN: track 91.8 -> 77.9 mm
- net Net-(JP1-Pad3): track 0.00 -> 13.0 mm
- net CB_D1: track 108.0 -> 119.2 mm
- net SCL: track 127.0 -> 116.4 mm
- net CB_D7: track 140.6 -> 131.5 mm
- net XCLK: track 95.7 -> 87.0 mm
- net CB_GND: track 45.2 -> 37.0 mm
- net PCLK: track 100.1 -> 93.4 mm
- net HREF: track 87.1 -> 93.6 mm
- net VS: track 108.3 -> 113.5 mm
- net CB_D0: track 104.2 -> 100.0 mm, vias 1 -> 2
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Other:
- board text added: "LED"
- board text added: "rev 0.0.3"
- board text removed: "P20"
- board text removed: "rev 0.0.2"
